File: BurnWire.kicad_sch (KiCad schematic)
At the start: 14 parts, among them J1 B6B-XH-A_LF__SN_, U1 ADP2303ARDZ

Commit message: updated schematic
Parts:
- removed C5: WCAP-ASLI_5X5.5, WCAP-ASLI:WCAP-ASLI_5X5.5_DXL_, symbol WCAP-ASLI_5X5.5:WCAP-ASLI_5X5.5
- removed L1: NLV32T-3R3J-EF, imported_footprints:IND_NLV32T_TDK, symbol 2025-11-02_20-08-03:NLV32T-3R3J-EF
- removed TP1, TP2: TestPoint_Alt, TestPoint:TestPoint_2Pads_Pitch5.08mm_Drill1.3mm, symbol Connector:TestPoint_Alt
- added L1: SRN6045-3R3Y, IND_BOURNS_SRN6045, symbol 2026-04-05_19-15-18:SRN6045-3R3Y
- R1: value 10K -> 10k; footprint Resistor_THT:R_Axial_DIN0204_L3.6mm_D1.6mm_P2.54mm_Vertical -> (none)
- R2: value 0.5 -> 10k; footprint Resistor_THT:R_Axial_DIN0204_L3.6mm_D1.6mm_P5.08mm_Horizontal -> (none)
- R3: value 10K -> 100K
Connections:
- net VBatt is gone; now on net EN: C2.1, J1.1, R3.1, U1.2 (Vin)
- net VCutN: no longer R1.2, R2.1
- net Vout: now also R1.1, L1.1
- net at U1.5 (FB): now also R1.2, R2.1; no longer R1.1
- net at C1.2, CR1.1, U1.8 (SW): now also L1.2
Other:
- moved on the sheet: C2, C3, C4, CR1, R3

Commit message: Polished schema w/ labels, test points; updated layout for new Vout->FB VDivider
Parts:
- added TP1, TP2: TestPoint_Alt, symbol Connector:TestPoint_Alt
- renumbered R2 to RBott, R1 to RTop
Connections:
- net VCutN: now also RBott.1, RTop.2, U1.5 (FB), TP2.1
- net BST: now reaches C1.1, U1.1 (BST)
- net PGOOD: now reaches J1.5, R3.2, U1.4 (PGOOD)
- net SW: now reaches C1.2, CR1.1, L1.2, U1.8 (SW)
- net SW: now also TP1.1
Changed lines of the file:
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@@
+	)
+	(junction
+		(at 162.56 95.25)
+		(diameter 0)
+		(color 0 0 0 0)
 	)
 	(junction
@@
 	(wire
 		(pts
+			(xy 162.56 95.25) (xy 200.66 95.25)
+		)
+		(stroke
+			(width 0)
+			(type default)
+		)
+	)
+	(wire
+		(pts
 			(xy 194.31 71.12) (xy 194.31 69.85)
 		)
@@
 	(wire
 		(pts
+			(xy 162.56 95.25) (xy 162.56 92.71)
+		)
+		(stroke
+			(width 0)
+			(type default)
+		)
+	)
+	(wire
+		(pts
 			(xy 80.01 87.63) (xy 83.82 87.63)
 		)
@@
 	(wire
 		(pts
-			(xy 200.66 95.25) (xy 130.81 95.25)
+			(xy 130.81 95.25) (xy 162.56 95.25)
+		)
+		(stroke
+			(width 0)
+			(type default)
+		)
+	)
+	(wire
+		(pts
+			(xy 139.7 82.55) (xy 139.7 85.09)
 		)
 		(stroke
@@
 		)
 	)
-	(label "VCutN"
-		(at 143.51 87.63 0)
-		(effects
-			(font
-				(size 1.27 1.27)
-			)
-			(justify left bottom)
-		)
-	)
 	(label "VBatt"
 		(at 86.36 119.38 0)
@@
 		)
 	)
+	(label "PGOOD"
+		(at 78.74 106.68 0)
+		(effects
+			(font
+				(size 1.27 1.27)
+			)
+			(justify left bottom)
+		)
+	)
+	(label "BST"
+		(at 129.54 67.31 0)
+		(effects
+			(font
+				(size 1.27 1.27)
+			)
+			(justify left bottom)
+		)
+	)
 	(label "EN"
 		(at 80.01 127 0)
@@
 	(label "VCutN"
 		(at 80.01 124.46 0)
+		(effects
+			(font
+				(size 1.27 1.27)
+			)
+			(justify left bottom)
+		)
+	)
+	(label "SW"
+		(at 139.7 82.55 0)
+		(effects
+			(font
+				(size 1.27 1.27)
+			)
+			(justify left bottom)
+		)
+	)
+	(label "VCutN"
+		(at 130.81 88.9 0)
 		(effects
 			(font
@@
 	)
 	(symbol
+		(lib_id "Connector:TestPoint_Alt")
+		(at 162.56 92.71 0)
+		(unit 1)
+		(exclude_from_sim no)
+		(in_bom yes)
+		(on_board yes)
+		(dnp no)
+		(fields_autoplaced yes)
+		(property "Reference" "TP2"
+			(at 165.1 88.1379 0)
+			(effects
+				(font
+					(size 1.27 1.27)
+				)
+				(justify left)
+			)
+		)
+		(property "Value" "TestPoint_Alt"
+			(at 165.1 90.6779 0)
+			(effects
+				(font
+					(size 1.27 1.27)
+				)
+				(justify left)
+			)
+		)
+		(property "Footprint" ""
+			(at 167.64 92.71 0)
+			(effects
+				(font
+					(size 1.27 1.27)
+				)
+				(hide yes)
+			)
+		)
+		(property "Datasheet" "~"
+			(at 167.64 92.71 0)
+			(effects
+				(font
+					(size 1.27 1.27)
+				)
+				(hide yes)
+			)
+		)
+		(property "Description" "test point (alternative shape)"
+			(at 162.56 92.71 0)
+			(effects
+				(font
+					(size 1.27 1.27)
+				)
+				(hide yes)
+			)
+		)
+		(pin "1"
+		)
+		(instances
+			(project ""
+				(path "/f35490b1-adcb-463e-9dac-9bc4e552c2ef"
+					(reference "TP2")
+					(unit 1)
+				)
+			)
+		)
+	)
+	(symbol
 		(lib_id "Device:C_Small")
 		(at 139.7 74.93 0)
@@
 		(dnp no)
 		(fields_autoplaced yes)
-		(property "Reference" "R1"
+		(property "Reference" "RTop"
 			(at 203.2 87.6299 0)
 			(effects
@@
 			(project ""
 				(path "/f35490b1-adcb-463e-9dac-9bc4e552c2ef"
-					(reference "R1")
+					(reference "RTop")
 					(unit 1)
 				)
@@
 	)
 	(symbol
+		(lib_id "Connector:TestPoint_Alt")
+		(at 139.7 85.09 180)
+		(unit 1)
+		(exclude_from_sim no)
+		(in_bom yes)
+		(on_board yes)
+		(dnp no)
+		(fields_autoplaced yes)
+		(property "Reference" "TP1"
+			(at 142.24 87.1219 0)
+			(effects
+				(font
+					(size 1.27 1.27)
+				)
+				(justify right)
+			)
+		)
+		(property "Value" "TestPoint_Alt"
+			(at 142.24 89.6619 0)
+			(effects
+				(font
+					(size 1.27 1.27)
+				)
+				(justify right)
+			)
+		)
+		(property "Footprint" ""
+			(at 134.62 85.09 0)
+			(effects
+				(font
+					(size 1.27 1.27)
+				)
+				(hide yes)
+			)
+		)
+		(property "Datasheet" "~"
+			(at 134.62 85.09 0)
+			(effects
+				(font
+					(size 1.27 1.27)
+				)
+				(hide yes)
+			)
+		)
+		(property "Description" "test point (alternative shape)"
+			(at 139.7 85.09 0)
+			(effects
+				(font
+					(size 1.27 1.27)
+				)
+				(hide yes)
+			)
+		)
+		(pin "1"
+		)
+		(instances
+			(project ""
+				(path "/f35490b1-adcb-463e-9dac-9bc4e552c2ef"
+					(reference "TP1")
+					(unit 1)
+				)
+			)
+		)
+	)
+	(symbol
 		(lib_id "Device:R_US")
 		(at 200.66 101.6 0)
@@
 		(dnp no)
 		(fields_autoplaced yes)
-		(property "Reference" "R2"
+		(property "Reference" "RBott"
 			(at 203.2 100.3299 0)
 			(effects
@@
 			(project ""
 				(path "/f35490b1-adcb-463e-9dac-9bc4e552c2ef"
-					(reference "R2")
+					(reference "RBott")
 					(unit 1)
 				)

Commit message: added kiran schematic
Parts:
- removed C1: 0.1uF, Capacitor_THT:CP_Axial_L10.0mm_D4.5mm_P15.00mm_Horizontal, symbol Device:C_Small
- removed C2: 10uF, Capacitor_THT:CP_Axial_L10.0mm_D4.5mm_P15.00mm_Horizontal, symbol Device:C_Small
- removed C3, C4: WCAP-ASLI_5X5.5, WCAP-ASLI:WCAP-ASLI_5X5.5_DXL_, symbol WCAP-ASLI_5X5.5:WCAP-ASLI_5X5.5
- removed CR1: B330B-13-F, imported_footprints:CR_SMB_320-345BE_DIO, symbol 2025-11-01_22-47-16:B330B-13-F
- removed J1: B6B-XH-A_LF__SN_, imported_footprints:JST_B6B-XH-A_LF__SN_, symbol B6B-XH-A_LF__SN_:B6B-XH-A_LF__SN_
- removed L1: SRN6045-3R3Y, IND_BOURNS_SRN6045, symbol 2026-04-05_19-15-18:SRN6045-3R3Y
- removed RBott, RTop: 10k, symbol Device:R_US
- removed TP1, TP2: TestPoint_Alt, symbol Connector:TestPoint_Alt
- added C1, C2, C3, C4: C_US, symbol Device:C_US
- added D1: MBRS340, Diode_SMD:D_SMC, symbol Diode:MBRS340
- added J1, J2: Conn_01x02, symbol Connector_Generic:Conn_01x02
- added L1: L, symbol Device:L
- added R1, R2, R4: R_US, symbol Device:R_US
- R3: value 100K -> R_US; footprint Resistor_THT:R_Axial_DIN0204_L3.6mm_D1.6mm_P5.08mm_Horizontal -> (none)
Connections:
- net SW is gone; now on an unnamed net: U1.8 (SW)
- net VCutN is gone; now on an unnamed net: U1.5 (FB)
- net GND: now also R3.1, U1.4 (PGOOD), C1.2, C3.1, C3.2, C4.1, C4.2, D1.2 (A), J1.1 (Pin_1), J1.2 (Pin_2), J2.2 (Pin_2), L1.2, R2.2, R4.2
- net BST: no longer names the net of U1.1 (BST)
- net BST: now also C2.1
- removed net EN: R3.1, U1.2 (Vin), U1.3 (EN)
- net PGOOD: no longer names the net of R3.2
- net PGOOD: now also C2.2, D1.1 (K), L1.1, R4.1; no longer U1.4 (PGOOD)
- new net: R1.2, R2.1, U1.3 (EN)
- new net: C1.1, J2.1 (Pin_1), R1.1, U1.2 (Vin)
