File: Burn Wire Dev Board.kicad_sch (KiCad schematic)
At the start: 24 parts, among them J1 282834-2, J2 J-TSM-106-01-F-SV, J3 J-0532610671, U2 ADP2303ARDZ

Commit message: current sensor added to schematic forgot to save
Parts:
- added R4: 1k, symbol Device:R_US
- renumbered R2 to R1, R3 to R2, R4 to R3, U2 to U1
Connections:
- net BURN_NEG: now also R4.1
- new net TO_COMPUTE: R4.2
Other:
- moved on the sheet: R2, R3, TP2

Commit message: added compute resistor tolayout
Parts:
- removed D1: B540C-13-F, burn_wire:CR_SMB_320-345BE_DIO-L, symbol Burn Wire Dev Board:root_3_D-B540C-13-F_Burn Wire Dev Board.SchLib
- removed J2: J-TSM-106-01-F-SV, Connector_PinHeader_2.54mm:PinHeader_1x06_P2.54mm_Vertical, symbol Burn Wire Dev Board:root_0_mirrored_J-TSM-106-01-F-SV_Burn Wire Dev Board.SchLib
- removed J3: J-0532610671, Connector_PinHeader_2.54mm:PinHeader_1x08_P2.54mm_Vertical, symbol Burn Wire Dev Board:root_0_J-0532610671_Burn Wire Dev Board.SchLib
- added D1: D_Schottky, burn_wire:CR_SMB_320-345BE_DIO-L, symbol Device:D_Schottky
- added J1: Conn_01x06_Pin, Connector_PinSocket_2.54mm:PinSocket_1x06_P2.54mm_Vertical, symbol Connector:Conn_01x06_Pin
- added J3: Conn_01x02_Pin, Connector_PinSocket_2.54mm:PinSocket_1x02_P2.54mm_Vertical, symbol Connector:Conn_01x02_Pin
- added J4: Conn_01x01_Pin, Connector_PinSocket_2.54mm:PinSocket_1x01_P2.54mm_Horizontal, symbol Connector:Conn_01x01_Pin
- L1: ALTIUM_VALUE 6.8 uH -> 3.3uH
- R3: footprint Resistor_SMD:R_2010_5025Metric -> Resistor_SMD:R_2512_6332Metric
- R4: footprint (none) -> Resistor_SMD:R_0805_2012Metric_Pad1.20x1.40mm_HandSolder
- R5, R6: footprint Resistor_SMD:R_0805_2012Metric_Pad1.20x1.40mm_HandSolder -> Resistor_SMD:R_0603_1608Metric_Pad0.98x0.95mm_HandSolder
- renumbered J1 to J2
Connections:
- net BURN_NEG: now also J3.1 (Pin_1)
- net BURN_POS: now also J3.2 (Pin_2)
- net ENABLE: now also J1.1 (Pin_1)
- net GND: now also D1.1 (K), J1.4 (Pin_4), J1.5 (Pin_5), J1.6 (Pin_6)
- net PGOOD: now also J1.3 (Pin_3)
- net TO_COMPUTE: now also J4.1 (Pin_1)
- net at C2.1, L1.2, U1.8 (SW): now also D1.2 (A)
- net +5 renamed +VBATT
- net +VBATT: now also J1.2 (Pin_2)
Other:
- moved on the sheet: C3, C4, C5, L1
